Commit message: added meshes to simplified package to remove dependency on walkernew package

File: src/simplified/solidModel.urdf.xacro (robot description, xacro)
@@ -28,5 +28,5 @@
     <origin xyz="${(-27*inch)-forward_leg_extension} ${-1.6*inch} ${(14.63+1.75)*inch}" rpy="${M_PI/2+0.12} 0 ${-M_PI/2-0.06}" />
     <geometry>
-     <mesh filename="package://walkernew/meshes/Left Front Leg Revised 2.STL" scale="0.001 0.001 0.001"/>
+     <mesh filename="package://simplified/meshes/Left Front Leg Revised 2.STL" scale="0.001 0.001 0.001"/>
     </geometry>
      <material name="red">
@@ -37,5 +37,5 @@
      <origin xyz="${(-27*inch)-forward_leg_extension} ${-1.6*inch} ${(14.63+1.75)*inch}" rpy="${M_PI/2+0.12} 0 ${-M_PI/2-0.06}" />
     <geometry>
-     <mesh filename="package://walkernew/meshes/Left Front Leg Revised 2.STL" scale="0.001 0.001 0.001"/>
+     <mesh filename="package://simplified/meshes/Left Front Leg Revised 2.STL" scale="0.001 0.001 0.001"/>
     </geometry>
     </collision>
@@ -50,5 +50,5 @@
     <origin xyz="${backwards_leg_extension} 0 ${17.8*inch}" rpy="0.025 0.41 ${M_PI/2}" />
     <geometry>
-     <mesh filename="package://walkernew/meshes/Back Left Leg Revised 2.STL" scale="0.001 0.001 0.001"/>
+     <mesh filename="package://simplified/meshes/Back Left Leg Revised 2.STL" scale="0.001 0.001 0.001"/>
     </geometry>
      <material name="red">
@@ -59,5 +59,5 @@
    <origin xyz="0 0 ${17.8*inch}" rpy="0.025 0.41 ${M_PI/2}" />
     <geometry>
-     <mesh filename="package://walkernew/meshes/Back Left Leg Revised 2.STL" scale="0.001 0.001 0.001"/>
+     <mesh filename="package://simplified/meshes/Back Left Leg Revised 2.STL" scale="0.001 0.001 0.001"/>
     </geometry>
     </collision>
@@ -72,5 +72,5 @@
     <origin xyz="0 0 ${18.35*inch}" rpy="${M_PI/2} 0 0" />
     <geometry>
-     <mesh filename="package://walkernew/meshes/CoreToLeg.STL" scale="0.001 0.001 0.001"/>
+     <mesh filename="package://simplified/meshes/CoreToLeg.STL" scale="0.001 0.001 0.001"/>
     </geometry>
      <material name="red">
@@ -81,5 +81,5 @@
      <origin xyz="0 0 ${18.35*inch}" rpy="${M_PI/2} 0 0" />
     <geometry>
-     <mesh filename="package://walkernew/meshes/CoreToLeg.STL" scale="0.001 0.001 0.001"/>
+     <mesh filename="package://simplified/meshes/CoreToLeg.STL" scale="0.001 0.001 0.001"/>
     </geometry>
     </collision>
@@ -94,5 +94,5 @@
     <origin xyz="0 0 ${31*inch}" rpy="${M_PI/2} ${3*M_PI/2} 0" />
     <geometry>
-     <mesh filename="package://walkernew/meshes/Core Revised.STL" scale="0.001 0.001 0.001"/>
+     <mesh filename="package://simplified/meshes/Core Revised.STL" scale="0.001 0.001 0.001"/>
     </geometry>
      <material name="red">
@@ -103,5 +103,5 @@
     <origin xyz="0 0 ${31*inch}" rpy="${M_PI/2} ${3*M_PI/2} 0" />
     <geometry>
-     <mesh filename="package://walkernew/meshes/Core Revised.STL" scale="0.001 0.001 0.001"/>
+     <mesh filename="package://simplified/meshes/Core Revised.STL" scale="0.001 0.001 0.001"/>
     </geometry>
     </collision>
@@ -131,5 +131,5 @@
     <origin xyz="0 0 ${21.75*inch}" rpy="${M_PI/2} 0 0" />
     <geometry>
-     <mesh filename="package://walkernew/meshes/HandleBottom.STL" scale="0.001 0.001 0.001"/>
+     <mesh filename="package://simplified/meshes/HandleBottom.STL" scale="0.001 0.001 0.001"/>
     </geometry>
      <material name="red">
@@ -140,5 +140,5 @@
    <origin xyz="0 0 ${21.75*inch}" rpy="${M_PI/2} 0 0" />
     <geometry>
-     <mesh filename="package://walkernew/meshes/HandleBottom.STL" scale="0.001 0.001 0.001"/>
+     <mesh filename="package://simplified/meshes/HandleBottom.STL" scale="0.001 0.001 0.001"/>
     </geometry>
     </collision>
@@ -158,5 +158,5 @@
     <origin xyz="0 0 ${13.75*inch+handle_height}" rpy="${M_PI/2} 0 ${3*M_PI/2}" />
     <geometry>
-     <mesh filename="package://walkernew/meshes/Handle Revised.STL" scale="0.001 0.001 0.001"/>
+     <mesh filename="package://simplified/meshes/Handle Revised.STL" scale="0.001 0.001 0.001"/>
     </geometry>
      <material name="red">
@@ -167,5 +167,5 @@
    <origin xyz="0 0 ${13.75*inch+handle_height}" rpy="${M_PI/2} 0 ${3*M_PI/2}" />
     <geometry>
-     <mesh filename="package://walkernew/meshes/Handle Revised.STL" scale="0.001 0.001 0.001"/>
+     <mesh filename="package://simplified/meshes/Handle Revised.STL" scale="0.001 0.001 0.001"/>
     </geometry>
     </collision>
@@ -185,5 +185,5 @@
     <origin xyz="0 0 ${18.35*inch}" rpy="${3*M_PI/2} ${M_PI} 0" />
     <geometry>
-     <mesh filename="package://walkernew/meshes/CoreToLeg.STL" scale="0.001 0.001 0.001"/>
+     <mesh filename="package://simplified/meshes/CoreToLeg.STL" scale="0.001 0.001 0.001"/>
     </geometry>
      <material name="red">
@@ -194,5 +194,5 @@
    <origin xyz="0 0 ${18.35*inch}" rpy="${3*M_PI/2} ${M_PI} 0" />
     <geometry>
-     <mesh filename="package://walkernew/meshes/CoreToLeg.STL" scale="0.001 0.001 0.001"/>
+     <mesh filename="package://simplified/meshes/CoreToLeg.STL" scale="0.001 0.001 0.001"/>
     </geometry>
     </collision>
@@ -212,5 +212,5 @@
     <origin xyz="0 0 ${21.75*inch}" rpy="${3*M_PI/2} ${M_PI} 0" />
     <geometry>
-     <mesh filename="package://walkernew/meshes/HandleBottom.STL" scale="0.001 0.001 0.001"/>
+     <mesh filename="package://simplified/meshes/HandleBottom.STL" scale="0.001 0.001 0.001"/>
     </geometry>
      <material name="red">
@@ -221,5 +221,5 @@
      <origin xyz="0 0 ${21.75*inch}" rpy="${3*M_PI/2} ${M_PI} 0" />
     <geometry>
-     <mesh filename="package://walkernew/meshes/HandleBottom.STL" scale="0.001 0.001 0.001"/>
+     <mesh filename="package://simplified/meshes/HandleBottom.STL" scale="0.001 0.001 0.001"/>
     </geometry>
     </collision>
@@ -239,5 +239,5 @@
     <origin xyz="0 0 ${13.75*inch+handle_height}" rpy="${M_PI/2} 0 ${3*M_PI/2}" />
     <geometry>
-     <mesh filename="package://walkernew/meshes/Handle Revised.STL"
+     <mesh filename="package://simplified/meshes/Handle Revised.STL"
 scale="0.001 0.001 0.001"/>
     </geometry>
@@ -249,5 +249,5 @@
     <origin xyz="0 0 ${13.75*inch+handle_height}" rpy="${M_PI/2} 0 ${3*M_PI/2}" />
     <geometry>
-     <mesh filename="package://walkernew/meshes/Handle Revised.STL"
+     <mesh filename="package://simplified/meshes/Handle Revised.STL"
 scale="0.001 0.001 0.001"/>
     </geometry>
@@ -268,5 +268,5 @@
     <origin xyz="${2.75*inch-forward_leg_extension} ${0*inch} ${(14.63+1.75)*inch}" rpy="${M_PI/2+0.12} 0 ${-M_PI/2-0.06}" />
     <geometry>
-     <mesh filename="package://walkernew/meshes/Right Front Leg Revised 2.STL" scale="0.001 0.001 0.001"/>
+     <mesh filename="package://simplified/meshes/Right Front Leg Revised 2.STL" scale="0.001 0.001 0.001"/>
     </geometry>
      <material name="red">
@@ -277,5 +277,5 @@
     <origin xyz="${2.75*inch-forward_leg_extension} ${0*inch} ${(14.63+1.75)*inch}" rpy="${M_PI/2+0.12} 0 ${-M_PI/2-0.06}" />
     <geometry>
-     <mesh filename="package://walkernew/meshes/Right Front Leg Revised 2.STL" scale="0.001 0.001 0.001"/>
+     <mesh filename="package://simplified/meshes/Right Front Leg Revised 2.STL" scale="0.001 0.001 0.001"/>
     </geometry>
     </collision>
@@ -300,5 +300,5 @@
     <origin xyz="${backwards_leg_extension} 0 ${17.8*inch}" rpy="0.025 0.41 ${M_PI/2}" />
     <geometry>
-     <mesh filename="package://walkernew/meshes/Right Back Leg Revised 2.STL" scale="0.001 0.001 0.001"/>
+     <mesh filename="package://simplified/meshes/Right Back Leg Revised 2.STL" scale="0.001 0.001 0.001"/>
     </geometry>
      <material name="red">
@@ -309,5 +309,5 @@
     <origin xyz="0 0 ${17.8*inch}" rpy="0.025 0.41 ${M_PI/2}" />
     <geometry>
-     <mesh filename="package://walkernew/meshes/Right Back Leg Revised 2.STL" scale="0.001 0.001 0.001"/>
+     <mesh filename="package://simplified/meshes/Right Back Leg Revised 2.STL" scale="0.001 0.001 0.001"/>
     </geometry>
     </collision>
@@ -330,5 +330,5 @@
     <origin xyz="0 0 0" rpy="0 0 ${M_PI}" />
     <geometry>
-     <mesh filename="package://walkernew/meshes/WheelSpinning.STL" scale="0.001 0.001 0.001"/>
+     <mesh filename="package://simplified/meshes/WheelSpinning.STL" scale="0.001 0.001 0.001"/>
     </geometry>
      <material name="red">
@@ -339,5 +339,5 @@
     <origin xyz="0 0 0" rpy="0 0 ${M_PI}" />
     <geometry>
-     <mesh filename="package://walkernew/meshes/WheelSpinning.STL" scale="0.001 0.001 0.001"/>
+     <mesh filename="package://simplified/meshes/WheelSpinning.STL" scale="0.001 0.001 0.001"/>
     </geometry>
      <material name="red">
@@ -363,5 +363,5 @@
     <origin xyz="0 0 0" rpy="0 0 ${M_PI}" />
     <geometry>
-     <mesh filename="package://walkernew/meshes/WheelSpinning.STL" scale="0.001 0.001 0.001"/>
+     <mesh filename="package://simplified/meshes/WheelSpinning.STL" scale="0.001 0.001 0.001"/>
     </geometry>
      <material name="red">
@@ -372,5 +372,5 @@
    <origin xyz="0 0 0" rpy="0 0 ${M_PI}" />
     <geometry>
-     <mesh filename="package://walkernew/meshes/WheelSpinning.STL" scale="0.001 0.001 0.001"/>
+     <mesh filename="package://simplified/meshes/WheelSpinning.STL" scale="0.001 0.001 0.001"/>
     </geometry>
     </collision>
@@ -401,5 +401,5 @@
     <origin xyz="0 0 ${-6*inch}" rpy="0 ${M_PI/2-0.06} 0" />
     <geometry>
-     <mesh filename="package://walkernew/meshes/Wheel Direction.STL" scale="0.001 0.001 0.001"/>
+     <mesh filename="package://simplified/meshes/Wheel Direction.STL" scale="0.001 0.001 0.001"/>
     </geometry>
      <material name="red">
@@ -410,5 +410,5 @@
     <origin xyz="0 0 ${-6*inch}" rpy="0 ${M_PI/2-0.06} 0" />
     <geometry>
-     <mesh filename="package://walkernew/meshes/Wheel Direction.STL" scale="0.001 0.001 0.001"/>
+     <mesh filename="package://simplified/meshes/Wheel Direction.STL" scale="0.001 0.001 0.001"/>
     </geometry>
     </collision>
@@ -423,5 +423,5 @@
     <origin xyz="0 0 ${-6*inch}" rpy="0 ${M_PI/2-0.06} 0" />
     <geometry>
-     <mesh filename="package://walkernew/meshes/Wheel Direction.STL" scale="0.001 0.001 0.001"/>
+     <mesh filename="package://simplified/meshes/Wheel Direction.STL" scale="0.001 0.001 0.001"/>
     </geometry>
      <material name="red">
@@ -432,5 +432,5 @@
     <origin xyz="0 0 ${-6*inch}" rpy="0 ${M_PI/2-0.06} 0" />
     <geometry>
-     <mesh filename="package://walkernew/meshes/Wheel Direction.STL" scale="0.001 0.001 0.001"/>
+     <mesh filename="package://simplified/meshes/Wheel Direction.STL" scale="0.001 0.001 0.001"/>
     </geometry>
     </collision>
@@ -461,5 +461,5 @@
     <origin xyz="0 0 0" rpy="0 0 ${M_PI}" />
     <geometry>
-     <mesh filename="package://walkernew/meshes/WheelSpinning.STL" scale="0.001 0.001 0.001"/>
+     <mesh filename="package://simplified/meshes/WheelSpinning.STL" scale="0.001 0.001 0.001"/>
     </geometry>
      <material name="red">
@@ -470,5 +470,5 @@
    <origin xyz="0 0 0" rpy="0 0 ${M_PI}" />
     <geometry>
-     <mesh filename="package://walkernew/meshes/WheelSpinning.STL" scale="0.001 0.001 0.001"/>
+     <mesh filename="package://simplified/meshes/WheelSpinning.STL" scale="0.001 0.001 0.001"/>
     </geometry>
     </collision>
@@ -483,5 +483,5 @@
     <origin xyz="0 0 0" rpy="0 0 ${M_PI}" />
     <geometry>
-     <mesh filename="package://walkernew/meshes/WheelSpinning.STL" scale="0.001 0.001 0.001"/>
+     <mesh filename="package://simplified/meshes/WheelSpinning.STL" scale="0.001 0.001 0.001"/>
     </geometry>
      <material name="red">
@@ -492,5 +492,5 @@
     <origin xyz="0 0 0" rpy="0 0 0" />
     <geometry>
-     <mesh filename="package://walkernew/meshes/WheelSpinning.STL" scale="0.001 0.001 0.001"/>
+     <mesh filename="package://simplified/meshes/WheelSpinning.STL" scale="0.001 0.001 0.001"/>
     </geometry>
     </collision>
