Commit message: attached encoder plugin in gazebo, cleaned up .xacro .launch and .world files

File: src/simplified/solidModel.urdf.xacro (robot description, xacro)
@@ -559,42 +559,42 @@
     <provideFeedback>true</provideFeedback>
   </gazebo>
-<joint name="camera_rgb_joint" type="fixed">
-      <origin xyz="${cam_px+2*inch} ${kinect_cam_py+9*inch} ${cam_pz+22.5*inch}" rpy="${cam_or} ${cam_op} ${cam_oy+M_PI}"/>
-      <parent link="core"/>
-      <child link="camera_rgb_frame" />
-    </joint>
-    <link name="camera_rgb_frame"/>
-    <joint name="camera_rgb_optical_joint" type="fixed">
-      <origin xyz="0 0 0" rpy="${-M_PI/2} 0 ${-M_PI/2}" />
-      <parent link="camera_rgb_frame" />
-      <child link="camera_rgb_optical_frame" />
-    </joint>
-    <link name="camera_rgb_optical_frame"/>
-    <joint name="camera_joint" type="fixed">
-      <origin xyz="-0.031 ${-kinect_cam_py} -0.016" rpy="0 0 0"/>
-      <parent link="camera_rgb_frame"/>
-      <child link="camera_link"/>
-    </joint>
-      <link name="camera_link">
-      <visual>
-       <origin xyz="0 0 0" rpy="0 0 ${M_PI/2}"/>
-        <geometry>
-         <mesh filename="package://turtlebot_description/meshes/sensors/kinect.dae"/>
-        </geometry>
-      </visual>
-  	  <collision>
-        <origin xyz="0.0 0.0 0.0" rpy="0 0 0"/>
-  	    <geometry>
-  	      <box size="0.07271 0.27794 0.073"/>
-  	    </geometry>
-  	  </collision>
-      <inertial>
-        <mass value="0.564" />
-        <origin xyz="0 0 0" />
-        <inertia ixx="0.003881243" ixy="0.0" ixz="0.0"
-                 iyy="0.000498940" iyz="0.0"
-                 izz="0.003879257" />
-      </inertial>
-    </link>
+  <joint name="camera_rgb_joint" type="fixed">
+    <origin xyz="${cam_px+2*inch} ${kinect_cam_py+9*inch} ${cam_pz+22.5*inch}" rpy="${cam_or} ${cam_op} ${cam_oy+M_PI}"/>
+    <parent link="core"/>
+    <child link="camera_rgb_frame" />
+  </joint>
+  <link name="camera_rgb_frame"/>
+  <joint name="camera_rgb_optical_joint" type="fixed">
+    <origin xyz="0 0 0" rpy="${-M_PI/2} 0 ${-M_PI/2}" />
+    <parent link="camera_rgb_frame" />
+    <child link="camera_rgb_optical_frame" />
+  </joint>
+  <link name="camera_rgb_optical_frame"/>
+  <joint name="camera_joint" type="fixed">
+    <origin xyz="-0.031 ${-kinect_cam_py} -0.016" rpy="0 0 0"/>
+    <parent link="camera_rgb_frame"/>
+    <child link="camera_link"/>
+  </joint>
+  <link name="camera_link">
+    <visual>
+     <origin xyz="0 0 0" rpy="0 0 ${M_PI/2}"/>
+      <geometry>
+       <mesh filename="package://turtlebot_description/meshes/sensors/kinect.dae"/>
+      </geometry>
+    </visual>
+    <collision>
+      <origin xyz="0.0 0.0 0.0" rpy="0 0 0"/>
+      <geometry>
+        <box size="0.07271 0.27794 0.073"/>
+      </geometry>
+    </collision>
+    <inertial>
+      <mass value="0.564" />
+      <origin xyz="0 0 0" />
+      <inertia ixx="0.003881243" ixy="0.0" ixz="0.0"
+               iyy="0.000498940" iyz="0.0"
+               izz="0.003879257" />
+    </inertial>
+  </link>
     <!-- The fixed joints & links below are usually published by static_transformers launched by the OpenNi launch
          files. However, for Gazebo simulation we need them, so we add them here.
@@ -612,101 +612,127 @@
 	</joint>
 	<link name="camera_depth_optical_frame"/>
-    <gazebo reference="camera_link">
-      <sensor type="depth" name="camera">
-        <always_on>true</always_on>
-        <update_rate>20.0</update_rate>
-        <camera>
-          <horizontal_fov>${70.0*M_PI/180.0}</horizontal_fov>
-          <image>
-            <format>R8G8B8</format>
-            <width>1920</width>
-            <height>1080</height>
-          </image>
-          <clip>
-            <near>0.05</near>
-            <far>8.0</far>
-          </clip>
-        </camera>
-        <plugin name="kinect_camera_controller" filename="libgazebo_ros_openni_kinect.so">
-          <cameraName>camera</cameraName>
-          <alwaysOn>true</alwaysOn>
-          <updateRate>10</updateRate>
-          <imageTopicName>rgb/image_raw</imageTopicName>
-          <depthImageTopicName>depth_registered/image_raw</depthImageTopicName>
-          <pointCloudTopicName>depth_registered/points</pointCloudTopicName>
-          <cameraInfoTopicName>rgb/camera_info</cameraInfoTopicName>
-          <depthImageCameraInfoTopicName>depth_registered/camera_info</depthImageCameraInfoTopicName>
-          <frameName>camera_depth_optical_frame</frameName>
-          <baseline>0.1</baseline>
-          <distortion_k1>0.0</distortion_k1>
-          <distortion_k2>0.0</distortion_k2>
-          <distortion_k3>0.0</distortion_k3>
-          <distortion_t1>0.0</distortion_t1>
-          <distortion_t2>0.0</distortion_t2>
-          <pointCloudCutoff>0.4</pointCloudCutoff>
-          <pointCloudCutoffMax>5.0</pointCloudCutoffMax>
-        </plugin>
-      </sensor>
-    </gazebo>
-<transmission name="right_turning_wheel">
-  <type>transmission_interface/SimpleTransmission</type>
-  <joint name="front_right_leg_to_turning_wheel">
-    <hardwareInterface>PositionJointInterface</hardwareInterface>
-  </joint>
-  <actuator name="right_turning_actuator">
-    <mechanicalReduction>1</mechanicalReduction>
-  </actuator>
-</transmission>
-<transmission name="left_turning_wheel">
-  <type>transmission_interface/SimpleTransmission</type>
-  <joint name="front_left_leg_to_turning_wheel">
-    <hardwareInterface>PositionJointInterface</hardwareInterface>
-  </joint>
-  <actuator name="left_turning_actuator">
-    <mechanicalReduction>1</mechanicalReduction>
-  </actuator>
-</transmission>
-<transmission name="right_spinning_wheel">
-  <type>transmission_interface/SimpleTransmission</type>
-  <joint name="front_right_turning_to_spinning">
-    <hardwareInterface>VelocityJointInterface</hardwareInterface>
-  </joint>
-  <actuator name="right_spinning_actuator">
-    <mechanicalReduction>1</mechanicalReduction>
-  </actuator>
-</transmission>
-<transmission name="left_spinning_wheel">
-  <type>transmission_interface/SimpleTransmission</type>
-  <joint name="front_left_turning_to_spinning">
-    <hardwareInterface>VelocityJointInterface</hardwareInterface>
-  </joint>
-  <actuator name="left_spinning_actuator">
-    <mechanicalReduction>1</mechanicalReduction>
-  </actuator>
-</transmission>
-<transmission name="back_right_spinning_wheel">
-  <type>transmission_interface/SimpleTransmission</type>
-  <joint name="back_right_leg_to_wheel">
-    <hardwareInterface>EffortJointInterface</hardwareInterface>
-  </joint>
-  <actuator name="back_right_spinning_actuator">
-    <mechanicalReduction>1</mechanicalReduction>
-  </actuator>
-</transmission>
-<transmission name="back_left_spinning_wheel">
-  <type>transmission_interface/SimpleTransmission</type>
-  <joint name="back_left_leg_to_wheel">
-    <hardwareInterface>EffortJointInterface</hardwareInterface>
-  </joint>
-  <actuator name="back_left_spinning_actuator">
-    <mechanicalReduction>1</mechanicalReduction>
-  </actuator>
-</transmission>
-<link name="base_footprint">
-  <origin xyz="0 0 0" rpy="0 0 ${M_PI}" />
-</link>
-<joint name="base_joint" type="fixed">
-<parent link="base_footprint"/>
-<child link="core"/>
-</joint>
+  <gazebo reference="camera_link">
+    <sensor type="depth" name="camera">
+      <always_on>true</always_on>
+      <update_rate>20.0</update_rate>
+      <camera>
+        <horizontal_fov>${70.0*M_PI/180.0}</horizontal_fov>
+        <image>
+          <format>R8G8B8</format>
+          <width>1920</width>
+          <height>1080</height>
+        </image>
+        <clip>
+          <near>0.05</near>
+          <far>8.0</far>
+        </clip>
+      </camera>
+      <plugin name="kinect_camera_controller" filename="libgazebo_ros_openni_kinect.so">
+        <cameraName>camera</cameraName>
+        <alwaysOn>true</alwaysOn>
+        <updateRate>10</updateRate>
+        <imageTopicName>rgb/image_raw</imageTopicName>
+        <depthImageTopicName>depth_registered/image_raw</depthImageTopicName>
+        <pointCloudTopicName>depth_registered/points</pointCloudTopicName>
+        <cameraInfoTopicName>rgb/camera_info</cameraInfoTopicName>
+        <depthImageCameraInfoTopicName>depth_registered/camera_info</depthImageCameraInfoTopicName>
+        <frameName>camera_depth_optical_frame</frameName>
+        <baseline>0.1</baseline>
+        <distortion_k1>0.0</distortion_k1>
+        <distortion_k2>0.0</distortion_k2>
+        <distortion_k3>0.0</distortion_k3>
+        <distortion_t1>0.0</distortion_t1>
+        <distortion_t2>0.0</distortion_t2>
+        <pointCloudCutoff>0.4</pointCloudCutoff>
+        <pointCloudCutoffMax>5.0</pointCloudCutoffMax>
+      </plugin>
+    </sensor>
+  </gazebo>
+  <transmission name="right_turning_wheel">
+    <type>transmission_interface/SimpleTransmission</type>
+    <joint name="front_right_leg_to_turning_wheel">
+      <hardwareInterface>PositionJointInterface</hardwareInterface>
+    </joint>
+    <actuator name="right_turning_actuator">
+      <mechanicalReduction>1</mechanicalReduction>
+    </actuator>
+  </transmission>
+  <transmission name="left_turning_wheel">
+    <type>transmission_interface/SimpleTransmission</type>
+    <joint name="front_left_leg_to_turning_wheel">
+      <hardwareInterface>PositionJointInterface</hardwareInterface>
+    </joint>
+    <actuator name="left_turning_actuator">
+      <mechanicalReduction>1</mechanicalReduction>
+    </actuator>
+  </transmission>
+  <transmission name="right_spinning_wheel">
+    <type>transmission_interface/SimpleTransmission</type>
+    <joint name="front_right_turning_to_spinning">
+      <hardwareInterface>VelocityJointInterface</hardwareInterface>
+    </joint>
+    <actuator name="right_spinning_actuator">
+      <mechanicalReduction>1</mechanicalReduction>
+    </actuator>
+  </transmission>
+  <transmission name="left_spinning_wheel">
+    <type>transmission_interface/SimpleTransmission</type>
+    <joint name="front_left_turning_to_spinning">
+      <hardwareInterface>VelocityJointInterface</hardwareInterface>
+    </joint>
+    <actuator name="left_spinning_actuator">
+      <mechanicalReduction>1</mechanicalReduction>
+    </actuator>
+  </transmission>
+  <transmission name="back_right_spinning_wheel">
+    <type>transmission_interface/SimpleTransmission</type>
+    <joint name="back_right_leg_to_wheel">
+      <hardwareInterface>EffortJointInterface</hardwareInterface>
+    </joint>
+    <actuator name="back_right_spinning_actuator">
+      <mechanicalReduction>1</mechanicalReduction>
+    </actuator>
+  </transmission>
+  <transmission name="back_left_spinning_wheel">
+    <type>transmission_interface/SimpleTransmission</type>
+    <joint name="back_left_leg_to_wheel">
+      <hardwareInterface>EffortJointInterface</hardwareInterface>
+    </joint>
+    <actuator name="back_left_spinning_actuator">
+      <mechanicalReduction>1</mechanicalReduction>
+    </actuator>
+  </transmission>
+  <link name="base_footprint">
+    <origin xyz="0 0 0" rpy="0 0 ${M_PI}" />
+  </link>
+  <joint name="base_joint" type="fixed">
+    <parent link="base_footprint"/>
+    <child link="core"/>
+  </joint>
+  <gazebo>
+    <plugin name="rearLeftWheel_encoder_plugin" filename="libwheel_encoder_plugin.so">
+      <joint_name>back_left_leg_to_wheel</joint_name>
+      <ticks_per_revolution>400</ticks_per_revolution>
+      <topic_name>walkernew/rearLeftEncoder</topic_name>
+      <reverse_direction>1</reverse_direction>
+    </plugin>
+    <plugin name="rearRightWheel_encoder_plugin" filename="libwheel_encoder_plugin.so">
+      <joint_name>back_right_leg_to_wheel</joint_name>
+      <ticks_per_revolution>400</ticks_per_revolution>
+      <topic_name>walkernew/rearRightEncoder</topic_name>
+      <reverse_direction>1</reverse_direction>
+    </plugin>
+    <plugin name="frontLeftWheel_encoder_plugin" filename="libwheel_encoder_plugin.so">
+      <joint_name>front_left_leg_to_turning_wheel</joint_name>
+      <ticks_per_revolution>400</ticks_per_revolution>
+      <topic_name>walkernew/frontLeftEncoder</topic_name>
+      <reverse_direction>1</reverse_direction>
+    </plugin>
+    <plugin name="frontRightWheel_encoder_plugin" filename="libwheel_encoder_plugin.so">
+      <joint_name>front_right_leg_to_turning_wheel</joint_name>
+      <ticks_per_revolution>400</ticks_per_revolution>
+      <topic_name>walkernew/frontRightEncoder</topic_name>
+      <reverse_direction>1</reverse_direction>
+    </plugin>
+  </gazebo>
 </robot>
