Commit message: Continuing setup of robot_localization module
 - added changes to solid model
   --> using new .STL files
   --> physics consts need to be adjusted
   --> cleaned up some stuff using xacro/macros
 - added launch files

File: src/simplified/configs/solidModel.urdf.xacro (robot description, xacro)
@@ -30,7 +30,4 @@
      <mesh filename="package://simplified/meshes/Left Front Leg Revised 2.STL" scale="0.001 0.001 0.001"/>
     </geometry>
-     <material name="red">
-      <color rgba="1 0.5 0.5 1"/>
-    </material>
  </visual>
     <collision>
@@ -52,7 +49,4 @@
      <mesh filename="package://simplified/meshes/Back Left Leg Revised 2.STL" scale="0.001 0.001 0.001"/>
     </geometry>
-     <material name="red">
-      <color rgba="1 0.5 0.5 1"/>
-    </material>
  </visual>
     <collision>
@@ -74,7 +68,4 @@
      <mesh filename="package://simplified/meshes/CoreToLeg.STL" scale="0.001 0.001 0.001"/>
     </geometry>
-     <material name="red">
-      <color rgba="1 0.5 0.5 1"/>
-    </material>
  </visual>
     <collision>
@@ -96,7 +87,4 @@
      <mesh filename="package://simplified/meshes/Core Revised.STL" scale="0.001 0.001 0.001"/>
     </geometry>
-     <material name="red">
-      <color rgba="1 0.5 0.5 1"/>
-    </material>
  </visual>
     <collision>
@@ -133,7 +121,4 @@
      <mesh filename="package://simplified/meshes/HandleBottom.STL" scale="0.001 0.001 0.001"/>
     </geometry>
-     <material name="red">
-      <color rgba="1 0.5 0.5 1"/>
-    </material>
  </visual>
     <collision>
@@ -160,7 +145,4 @@
      <mesh filename="package://simplified/meshes/Handle Revised.STL" scale="0.001 0.001 0.001"/>
     </geometry>
-     <material name="red">
-      <color rgba="1 0.5 0.5 1"/>
-    </material>
  </visual>
     <collision>
@@ -187,7 +169,4 @@
      <mesh filename="package://simplified/meshes/CoreToLeg.STL" scale="0.001 0.001 0.001"/>
     </geometry>
-     <material name="red">
-      <color rgba="1 0.5 0.5 1"/>
-    </material>
  </visual>
     <collision>
@@ -214,7 +193,4 @@
      <mesh filename="package://simplified/meshes/HandleBottom.STL" scale="0.001 0.001 0.001"/>
     </geometry>
-     <material name="red">
-      <color rgba="1 0.5 0.5 1"/>
-    </material>
  </visual>
     <collision>
@@ -242,7 +218,4 @@
 scale="0.001 0.001 0.001"/>
     </geometry>
-     <material name="red">
-      <color rgba="1 0.5 0.5 1"/>
-    </material>
  </visual>
     <collision>
@@ -270,7 +243,4 @@
      <mesh filename="package://simplified/meshes/Right Front Leg Revised 2.STL" scale="0.001 0.001 0.001"/>
     </geometry>
-     <material name="red">
-      <color rgba="1 0.5 0.5 1"/>
-    </material>
  </visual>
     <collision>
@@ -302,7 +272,4 @@
      <mesh filename="package://simplified/meshes/Right Back Leg Revised 2.STL" scale="0.001 0.001 0.001"/>
     </geometry>
-     <material name="red">
-      <color rgba="1 0.5 0.5 1"/>
-    </material>
  </visual>
     <collision>
@@ -330,18 +297,12 @@
     <origin xyz="0 0 0" rpy="0 0 ${M_PI}" />
     <geometry>
-     <mesh filename="package://simplified/meshes/WheelSpinning.STL" scale="0.001 0.001 0.001"/>
-    </geometry>
-     <material name="red">
-      <color rgba="1 0.5 0.5 1"/>
-    </material>
+     <mesh filename="package://simplified/meshes/wheel.STL" scale="0.001 0.001 0.001"/>
+    </geometry>
  </visual>
     <collision>
     <origin xyz="0 0 0" rpy="0 0 ${M_PI}" />
     <geometry>
-     <mesh filename="package://simplified/meshes/WheelSpinning.STL" scale="0.001 0.001 0.001"/>
-    </geometry>
-     <material name="red">
-      <color rgba="1 0.5 0.5 1"/>
-    </material>
+     <mesh filename="package://simplified/meshes/wheel.STL" scale="0.001 0.001 0.001"/>
+    </geometry>
     </collision>
     <inertial>
@@ -363,14 +324,11 @@
     <origin xyz="0 0 0" rpy="0 0 ${M_PI}" />
     <geometry>
-     <mesh filename="package://simplified/meshes/WheelSpinning.STL" scale="0.001 0.001 0.001"/>
-    </geometry>
-     <material name="red">
-      <color rgba="1 0.5 0.5 1"/>
-    </material>
+     <mesh filename="package://simplified/meshes/wheel.STL" scale="0.001 0.001 0.001"/>
+    </geometry>
  </visual>
     <collision>
    <origin xyz="0 0 0" rpy="0 0 ${M_PI}" />
     <geometry>
-     <mesh filename="package://simplified/meshes/WheelSpinning.STL" scale="0.001 0.001 0.001"/>
+     <mesh filename="package://simplified/meshes/wheel.STL" scale="0.001 0.001 0.001"/>
     </geometry>
     </collision>
@@ -381,12 +339,17 @@
     </inertial>
  </link>
+<!-- Front Wheel Yaw Joint Params -->
+<xacro:property name="front_yaw_effort_limit" value="100.0"/>
+<xacro:property name="front_yaw_velocity_limit" value="100.0"/>
+<xacro:property name="front_yaw_damping" value="0.5"/>
+<xacro:property name="front_yaw_friction" value="0.0"/>
 <joint name="front_right_leg_to_turning_wheel" type="continuous">
     <parent link="front_right_leg"/>
     <child link="front_right_turning_wheel"/>
     <origin xyz="${4.25*inch-forward_leg_extension} ${-2.4*inch} ${10*inch}"/>
-	<axis xyz="0 0 1"/>
-<limit effort="100" velocity="100.0"  />
-     <joint_properties damping="0.05" friction="0.05"/>
-  </joint>
+    <axis xyz="0 0 1"/>
+    <limit effort="${front_yaw_effort_limit}" velocity="${front_yaw_velocity_limit}"  />
+    <joint_properties damping="${front_yaw_damping}" friction="${front_yaw_friction}"/>
+</joint>
 <joint name="front_left_leg_to_turning_wheel" type="continuous">
     <parent link="front_left_leg"/>
@@ -394,21 +357,18 @@
     <axis xyz="0 0 1"/>
     <origin xyz="${-25.50*inch-forward_leg_extension} ${-2.4*inch} ${10*inch}"/>
-    <limit effort="100" velocity="100"/>
-     <joint_properties damping="0.05" friction="0.05"/>
-  </joint>
+    <limit effort="${front_yaw_effort_limit}" velocity="${front_yaw_velocity_limit}"  />
+    <joint_properties damping="${front_yaw_damping}" friction="${front_yaw_friction}"/>
+</joint>
 <link name="front_right_turning_wheel">
   <visual>
-    <origin xyz="0 0 ${-6*inch}" rpy="0 ${M_PI/2-0.06} 0" />
-    <geometry>
-     <mesh filename="package://simplified/meshes/Wheel Direction.STL" scale="0.001 0.001 0.001"/>
-    </geometry>
-     <material name="red">
-      <color rgba="1 0.5 0.5 1"/>
-    </material>
- </visual>
-    <collision>
-    <origin xyz="0 0 ${-6*inch}" rpy="0 ${M_PI/2-0.06} 0" />
-    <geometry>
-     <mesh filename="package://simplified/meshes/Wheel Direction.STL" scale="0.001 0.001 0.001"/>
+    <origin xyz="0 0 0" rpy="0 ${M_PI/2-0.06} 0" />
+    <geometry>
+     <mesh filename="package://simplified/meshes/frontwheelhub.STL" scale="0.001 0.001 0.001"/>
+    </geometry>
+ </visual>
+    <collision>
+    <origin xyz="0 0 0" rpy="0 ${M_PI/2-0.06} 0" />
+    <geometry>
+     <mesh filename="package://simplified/meshes/frontwheelhub.STL" scale="0.001 0.001 0.001"/>
     </geometry>
     </collision>
@@ -421,16 +381,13 @@
 <link name="front_left_turning_wheel">
   <visual>
-    <origin xyz="0 0 ${-6*inch}" rpy="0 ${M_PI/2-0.06} 0" />
-    <geometry>
-     <mesh filename="package://simplified/meshes/Wheel Direction.STL" scale="0.001 0.001 0.001"/>
-    </geometry>
-     <material name="red">
-      <color rgba="1 0.5 0.5 1"/>
-    </material>
- </visual>
-    <collision>
-    <origin xyz="0 0 ${-6*inch}" rpy="0 ${M_PI/2-0.06} 0" />
-    <geometry>
-     <mesh filename="package://simplified/meshes/Wheel Direction.STL" scale="0.001 0.001 0.001"/>
+    <origin xyz="0 0 0" rpy="0 ${M_PI/2-0.06} 0" />
+    <geometry>
+     <mesh filename="package://simplified/meshes/frontwheelhub.STL" scale="0.001 0.001 0.001"/>
+    </geometry>
+ </visual>
+    <collision>
+    <origin xyz="0 0 0" rpy="0 ${M_PI/2-0.06} 0" />
+    <geometry>
+     <mesh filename="package://simplified/meshes/frontwheelhub.STL" scale="0.001 0.001 0.001"/>
     </geometry>
     </collision>
@@ -441,11 +398,16 @@
     </inertial>
  </link>
+<!-- Front Wheel Rotational Joint Params -->
+<xacro:property name="front_rotational_effort_limit" value="100.0"/>
+<xacro:property name="front_rotational_velocity_limit" value="100.0"/>
+<xacro:property name="front_rotational_damping" value="0.1"/>
+<xacro:property name="front_rotational_friction" value="0.2"/>
 <joint name="front_right_turning_to_spinning" type="continuous">
     <parent link="front_right_turning_wheel"/>
     <child link="front_right_spinning_wheel"/>
     <axis xyz="0 1 0"/>
-    <origin xyz="0 ${0.65*inch} ${-6*inch}"/>
-     <limit effort="100" velocity="100"/>
-      <joint_properties damping="0.1" friction="0.2"/>
+    <origin xyz="0.04558 ${0.65*inch} ${-6*inch}"/>
+    <limit effort="${front_rotational_effort_limit}" velocity="${front_rotational_velocity_limit}"  />
+    <joint_properties damping="${front_rotational_damping}" friction="${front_rotational_friction}"/>
   </joint>
 <joint name="front_left_turning_to_spinning" type="continuous">
@@ -453,5 +415,5 @@
     <child link="front_left_spinning_wheel"/>
     <axis xyz="0 1 0"/>
-    <origin xyz="0 ${0.65*inch} ${-6*inch}"/>
+    <origin xyz="0.04558 ${0.65*inch} ${-6*inch}"/>
     <limit effort="100" velocity="100"/>
       <joint_properties damping="0.1" friction="0.2"/>
@@ -461,18 +423,15 @@
     <origin xyz="0 0 0" rpy="0 0 ${M_PI}" />
     <geometry>
-     <mesh filename="package://simplified/meshes/WheelSpinning.STL" scale="0.001 0.001 0.001"/>
-    </geometry>
-     <material name="red">
-      <color rgba="1 0.5 0.5 1"/>
-    </material>
- </visual>
+     <mesh filename="package://simplified/meshes/wheel.STL" scale="0.001 0.001 0.001"/>
+    </geometry>
+  </visual>
     <collision>
    <origin xyz="0 0 0" rpy="0 0 ${M_PI}" />
     <geometry>
-     <mesh filename="package://simplified/meshes/WheelSpinning.STL" scale="0.001 0.001 0.001"/>
-    </geometry>
-    </collision>
-    <inertial>
-    <origin xyz="0 0 0" rpy="0 0 0" />
+     <mesh filename="package://simplified/meshes/wheel.STL" scale="0.001 0.001 0.001"/>
+    </geometry>
+    </collision>
+    <inertial>
+    <origin xyz="0.04558 0 0" rpy="0 0 0" />
       <mass value="2.28"/>
       <inertia ixx="0.01" ixy="0" ixz="0" iyy="0.02" iyz="0" izz="0.01"/>
@@ -483,18 +442,15 @@
     <origin xyz="0 0 0" rpy="0 0 ${M_PI}" />
     <geometry>
-     <mesh filename="package://simplified/meshes/WheelSpinning.STL" scale="0.001 0.001 0.001"/>
-    </geometry>
-     <material name="red">
-      <color rgba="1 0.5 0.5 1"/>
-    </material>
+     <mesh filename="package://simplified/meshes/wheel.STL" scale="0.001 0.001 0.001"/>
+    </geometry>
  </visual>
     <collision>
     <origin xyz="0 0 0" rpy="0 0 0" />
     <geometry>
-     <mesh filename="package://simplified/meshes/WheelSpinning.STL" scale="0.001 0.001 0.001"/>
-    </geometry>
-    </collision>
-    <inertial>
-    <origin xyz="0 0 0" rpy="0 0 0" />
+     <mesh filename="package://simplified/meshes/wheel.STL" scale="0.001 0.001 0.001"/>
+    </geometry>
+    </collision>
+    <inertial>
+    <origin xyz="0.04558 0 0" rpy="0 0 0" />
       <mass value="2.28"/>
       <inertia ixx="0.01" ixy="0" ixz="0" iyy="0.02" iyz="0" izz="0.01"/>
@@ -515,48 +471,54 @@
     <provideFeedback>true</provideFeedback>
 </gazebo>
+<!-- Front Wheel Rotational Joint Params -->
+<xacro:property name="wheel_mu1" value="200"/>
+<xacro:property name="wheel_mu2" value="100"/>
+<xacro:property name="wheel_kp" value="1000000"/>
+<xacro:property name="wheel_kd" value="1"/>
+<xacro:property name="wheel_damping" value="0.50"/>
 <gazebo reference="front_left_spinning_wheel">
-    <mu1>0.99</mu1>
-    <mu2>0.9</mu2>
-    <kp>1000000</kp>
-    <kd>50</kd>
+    <mu1>${wheel_mu1}</mu1>
+    <mu2>${wheel_mu2}</mu2>
+    <kp>${wheel_kp}</kp>
+    <kd>${wheel_kd}</kd>
     <fdir1>1 0 0</fdir1>
     <gravity>true</gravity>
-    <dampingFactor>0.1</dampingFactor>
-    <material>Gazebo/Black</material>
-    <provideFeedback>true</provideFeedback>
-  </gazebo>
-<gazebo reference="back_right_spinning_wheel">
-    <mu1>0.99</mu1>
-    <mu2>0.9</mu2>
-    <kp>1000000</kp>
-    <kd>50</kd>
-    <fdir1>1 0 0</fdir1>
-    <gravity>true</gravity>
-    <dampingFactor>0.1</dampingFactor>
-    <material>Gazebo/Black</material>
-    <provideFeedback>true</provideFeedback>
-  </gazebo>
-<gazebo reference="back_left_spinning_wheel">
-    <mu1>0.99</mu1>
-    <mu2>0.9</mu2>
-    <kp>1000000</kp>
-    <kd>50</kd>
-    <fdir1>1 0 0</fdir1>
-    <gravity>true</gravity>
-    <dampingFactor>0.1</dampingFactor>
-    <material>Gazebo/Black</material>
+    <dampingFactor>${wheel_damping}</dampingFactor>
+    <material>Gazebo/Blue</material>
     <provideFeedback>true</provideFeedback>
   </gazebo>
 <gazebo reference="front_right_spinning_wheel">
-    <mu1>0.99</mu1>
-    <mu2>0.9</mu2>
-    <kp>1000000</kp>
-    <kd>50</kd>
+    <mu1>${wheel_mu1}</mu1>
+    <mu2>${wheel_mu2}</mu2>
+    <kp>${wheel_kp}</kp>
+    <kd>${wheel_kd}</kd>
     <fdir1>1 0 0</fdir1>
     <gravity>true</gravity>
-    <dampingFactor>0.1</dampingFactor>
+    <dampingFactor>${wheel_damping}</dampingFactor>
+    <material>Gazebo/Red</material>
+    <provideFeedback>true</provideFeedback>
+</gazebo>
+<gazebo reference="back_right_spinning_wheel">
+    <mu1>${wheel_mu1}</mu1>
+    <mu2>${wheel_mu2}</mu2>
+    <kp>${wheel_kp}</kp>
+    <kd>${wheel_kd}</kd>
+    <fdir1>1 0 0</fdir1>
+    <gravity>true</gravity>
+    <dampingFactor>${wheel_damping}</dampingFactor>
     <material>Gazebo/Black</material>
     <provideFeedback>true</provideFeedback>
-  </gazebo>
+</gazebo>
+<gazebo reference="back_left_spinning_wheel">
+    <mu1>${wheel_mu1}</mu1>
+    <mu2>${wheel_mu2}</mu2>
+    <kp>${wheel_kp}</kp>
+    <kd>${wheel_kd}</kd>
+    <fdir1>1 0 0</fdir1>
+    <gravity>true</gravity>
+    <dampingFactor>${wheel_damping}</dampingFactor>
+    <material>Gazebo/Black</material>
+    <provideFeedback>true</provideFeedback>
+</gazebo>
   <joint name="camera_rgb_joint" type="fixed">
     <origin xyz="${cam_px+2*inch} ${kinect_cam_py+9*inch} ${cam_pz+22.5*inch}" rpy="${cam_or} ${cam_op} ${cam_oy+M_PI}"/>

Commit message: cleaning up / adding docs / bug fixes
 - changed parameters in model urdf so that things are mostly workin
   - model doesn't drift
   - model doesn't break while driving
   - wheels don't appear to stutter while driving (encoder odometry should work somewhat now)
   - front wheel yaw joints are vibrating still
 - added some comments and a table of contents in urdf for quick *ctrl-f*ing
 - removed odometry.launch file as it was unneeded

File: src/simplified/configs/solidModel.urdf.xacro (robot description, xacro)
@@ -1,4 +1,17 @@
 <?xml version="1.0"?>
 <robot name="walkernew" xmlns:xacro="http://www.ros.org/wiki/xacro">
+<!-- Table of Contents - (ctrl-f to jump)
+Links:
+front left leg -               [FLL_L]
+back left leg  -               [BLL_L]
+core to left leg (link) -      [CTLL_L]
+core (link) -                  [CORE_L]
+handle left
+handle bottom left to handle
+front right turning wheel -    [FRTW_L]
+front left turning wheel -     [FLTW_L]
+front right spinning wheel -   [FRSW_L]
+front left spinning wheel -    [FLSW_L]
+-->
 <gazebo>
     <plugin name="gazebo_ros_control" filename="libgazebo_ros_control.so">
@@ -17,11 +30,12 @@
 	<property name="cam_op" value="0" />
 	<property name="cam_oy" value="0" />
- <origin xyz="0 0 0" rpy="0 0 0"/>
-<!-- List of Editable Walker Dimensions-->
-<property name="forward_leg_extension" value="${4*inch}" />
-<property name="backwards_leg_extension" value="${4*inch}" />
-<property name="frame_width" value="${3*inch}" />
-<property name="handle_width" value="${3*inch}" />
-<property name="handle_height" value="${5*inch}" />
+   <origin xyz="0 0 0" rpy="0 0 0"/>
+  <!-- List of Editable Walker Dimensions-->
+  <property name="forward_leg_extension" value="${4*inch}" />
+  <property name="backwards_leg_extension" value="${4*inch}" />
+  <property name="frame_width" value="${3*inch}" />
+  <property name="handle_width" value="${3*inch}" />
+  <property name="handle_height" value="${5*inch}" />
+<!-- [FLL_L] -->
 <link name="front_left_leg">
   <visual>
@@ -43,4 +57,5 @@
     </inertial>
  </link>
+<!-- [BLL_L] -->
 <link name="back_left_leg">
   <visual>
@@ -62,4 +77,5 @@
     </inertial>
  </link>
+<!-- [CTLL_L] -->
 <link name="core_to_leg_left">
   <visual>
@@ -81,4 +97,5 @@
     </inertial>
  </link>
+<!-- [CORE_L] -->
 <link name="core">
   <visual>
@@ -360,4 +377,5 @@
     <joint_properties damping="${front_yaw_damping}" friction="${front_yaw_friction}"/>
 </joint>
+<!-- [FRTW_L] -->
 <link name="front_right_turning_wheel">
   <visual>
@@ -368,15 +386,16 @@
  </visual>
     <collision>
-    <origin xyz="0 0 0" rpy="0 ${M_PI/2-0.06} 0" />
-    <geometry>
-     <mesh filename="package://simplified/meshes/frontwheelhub.STL" scale="0.001 0.001 0.001"/>
-    </geometry>
-    </collision>
-    <inertial>
-    <origin xyz="0 0 0" rpy="0 0 0" />
+      <origin xyz="0 0 0" rpy="0 ${M_PI/2-0.06} 0" />
+      <geometry>
+         <mesh filename="package://simplified/meshes/frontwheelhub.STL" scale="0.001 0.001 0.001"/>
+      </geometry>
+    </collision>
+    <inertial>
+      <origin xyz="0 0 0" rpy="0 0 0" />
       <mass value="0.79"/>
       <inertia ixx="0.01" ixy="0" ixz="0" iyy="0.01" iyz="0" izz="0"/>
     </inertial>
  </link>
+<!-- [FLTW_L] -->
 <link name="front_left_turning_wheel">
   <visual>
@@ -416,7 +435,8 @@
     <axis xyz="0 1 0"/>
     <origin xyz="0.04558 ${0.65*inch} ${-6*inch}"/>
-    <limit effort="100" velocity="100"/>
-      <joint_properties damping="0.1" friction="0.2"/>
-  </joint>
+    <limit effort="${front_rotational_effort_limit}" velocity="${front_rotational_velocity_limit}"  />
+    <joint_properties damping="${front_rotational_damping}" friction="${front_rotational_friction}"/>
+  </joint>
+<!-- [FRSW_L] -->
 <link name="front_right_spinning_wheel">
   <visual>
@@ -438,4 +458,5 @@
     </inertial>
  </link>
+<!-- [FLSW_L] -->
 <link name="front_left_spinning_wheel">
   <visual>
@@ -472,9 +493,9 @@
 </gazebo>
 <!-- Front Wheel Rotational Joint Params -->
-<xacro:property name="wheel_mu1" value="200"/>
-<xacro:property name="wheel_mu2" value="100"/>
+<xacro:property name="wheel_mu1" value="0.99"/>
+<xacro:property name="wheel_mu2" value="0.90"/>
 <xacro:property name="wheel_kp" value="1000000"/>
-<xacro:property name="wheel_kd" value="1"/>
-<xacro:property name="wheel_damping" value="0.50"/>
+<xacro:property name="wheel_kd" value="500000"/>
+<xacro:property name="wheel_damping" value="0.10"/>
 <gazebo reference="front_left_spinning_wheel">
     <mu1>${wheel_mu1}</mu1>
