Commit message: Whitespace changes only

File: src/simplified/configs/solidModel.urdf.xacro (robot description, xacro)
@@ -5,5 +5,5 @@
 Xacro Properties:
 Plugins:
-    Wheel Encoders:
+    Wheel Encoders Plugins         [WENC_P]
     Gazebo Ros Control (Joint Controllers):
 Links:
@@ -13,12 +13,26 @@
     Back Left Leg                  [BLL_L]
     Core to Left Leg (link)        [CTLL_L]
-    Core (link)                    [CORE_L]
-    Handle Left
-    Front Left Leg to Back Leg     [FLLTBL_L]
-    Handle Bottom Left to Handle
+    Handle Bottom Left             [HBL_L]
+    Handle Left                    [HL_L]
+    Core to Leg Right              [CTLR_L]
+    Handle Bottom Right            [HBR_L]
+    Handle Right                   [HR_L]
+    Front Right Leg                [FRL_L]
+    Back Right Leg                 [BRL_L]
+    Back Right Spinning Wheel      [BRSW_L]
+    Back Left Spinning Wheel       [BLSW_L]
     Front Right Turning Wheel      [FRTW_L]
     Front Left Turning Wheel       [FLTW_L]
     Front Right Spinning Wheel     [FRSW_L]
     Front Left Spinning Wheel      [FLSW_L]
+    Front Left Leg to Back Leg     [FLLTBL_L]
+    Handle Bottom Left to Handle
+Transmissions:
+    Right Turning Wheel            [RTW_T]
+    Left Turning Wheel             [LTW_T]
+    Right Spinning Wheel           [RSW_T]
+    Left Spinning Wheel            [LSW_T]
+    Back Right Spinning Wheel      [BRSW_T]
+    Back Left Spinning Wheel       [BLSW_T]
 -->
 <!-- PROPERTY LIST -->
@@ -153,23 +167,24 @@
     <origin xyz="${0.65*inch} ${-4*inch-(frame_width/2)} 0"/>
   </joint>
+<!-- Handle Bottom Left - [HBL_L] -->
 <link name="handle_bottom_left">
-  <visual>
-    <origin xyz="0 0 ${21.75*inch}" rpy="${M_PI/2} 0 0" />
-    <geometry>
-     <mesh filename="package://simplified/meshes/HandleBottom.STL" scale="0.001 0.001 0.001"/>
-    </geometry>
- </visual>
-    <collision>
-   <origin xyz="0 0 ${21.75*inch}" rpy="${M_PI/2} 0 0" />
-    <geometry>
-     <mesh filename="package://simplified/meshes/HandleBottom.STL" scale="0.001 0.001 0.001"/>
-    </geometry>
-    </collision>
-    <inertial>
-    <origin xyz="0 0.07 0.09" rpy="0 0 0" />
-      <mass value="0.5"/>
-      <inertia ixx="0.06" ixy="0" ixz="0" iyy="0.04" iyz="0" izz="0.02"/>
-    </inertial>
- </link>
+    <visual>
+        <origin xyz="0 0 ${21.75*inch}" rpy="${M_PI/2} 0 0" />
+        <geometry>
+            <mesh filename="package://simplified/meshes/HandleBottom.STL" scale="0.001 0.001 0.001"/>
+        </geometry>
+    </visual>
+    <collision>
+        <origin xyz="0 0 ${21.75*inch}" rpy="${M_PI/2} 0 0" />
+        <geometry>
+            <mesh filename="package://simplified/meshes/HandleBottom.STL" scale="0.001 0.001 0.001"/>
+        </geometry>
+    </collision>
+    <inertial>
+        <origin xyz="0 0.07 0.09" rpy="0 0 0" />
+        <mass value="0.5"/>
+        <inertia ixx="0.06" ixy="0" ixz="0" iyy="0.04" iyz="0" izz="0.02"/>
+    </inertial>
+</link>
 <joint name="core_to_bottom_handle_left" type="fixed">
     <parent link="core"/>
@@ -177,4 +192,5 @@
     <origin xyz="${0.7*inch} ${-2*inch-(handle_width/2)} 0"/>
   </joint>
+<!-- Handle Left - [HL_L] -->
 <link name="handle_left">
   <visual>
@@ -201,23 +217,24 @@
     <origin xyz="${1.5*inch} ${1.5*inch} 0"/>
   </joint>
+<!-- Core to Leg Right - [CTLR_L] -->
 <link name="core_to_leg_right">
-  <visual>
-    <origin xyz="0 0 ${18.35*inch}" rpy="${3*M_PI/2} ${M_PI} 0" />
-    <geometry>
-     <mesh filename="package://simplified/meshes/CoreToLeg.STL" scale="0.001 0.001 0.001"/>
-    </geometry>
- </visual>
-    <collision>
-   <origin xyz="0 0 ${18.35*inch}" rpy="${3*M_PI/2} ${M_PI} 0" />
-    <geometry>
-     <mesh filename="package://simplified/meshes/CoreToLeg.STL" scale="0.001 0.001 0.001"/>
-    </geometry>
-    </collision>
-    <inertial>
-    <origin xyz="0 -0.11 -0.02" rpy="0 0 0" />
-      <mass value="1.56"/>
-      <inertia ixx="0.03" ixy="0" ixz="0" iyy="0" iyz="0" izz="0.3"/>
-    </inertial>
- </link>
+    <visual>
+        <origin xyz="0 0 ${18.35*inch}" rpy="${3*M_PI/2} ${M_PI} 0" />
+        <geometry>
+            <mesh filename="package://simplified/meshes/CoreToLeg.STL" scale="0.001 0.001 0.001"/>
+        </geometry>
+    </visual>
+    <collision>
+        <origin xyz="0 0 ${18.35*inch}" rpy="${3*M_PI/2} ${M_PI} 0" />
+        <geometry>
+            <mesh filename="package://simplified/meshes/CoreToLeg.STL" scale="0.001 0.001 0.001"/>
+        </geometry>
+    </collision>
+    <inertial>
+        <origin xyz="0 -0.11 -0.02" rpy="0 0 0" />
+        <mass value="1.56"/>
+        <inertia ixx="0.03" ixy="0" ixz="0" iyy="0" iyz="0" izz="0.3"/>
+    </inertial>
+</link>
 <joint name="core_to_core_to_leg_right" type="fixed">
     <parent link="core"/>
@@ -225,23 +242,24 @@
     <origin xyz="${0.65*inch} ${20*inch+(frame_width/2)} 0"/>
   </joint>
+<!-- Handle Bottom Right - [HBR_L] -->
 <link name="handle_bottom_right">
-  <visual>
-    <origin xyz="0 0 ${21.75*inch}" rpy="${3*M_PI/2} ${M_PI} 0" />
-    <geometry>
-     <mesh filename="package://simplified/meshes/HandleBottom.STL" scale="0.001 0.001 0.001"/>
-    </geometry>
- </visual>
-    <collision>
-     <origin xyz="0 0 ${21.75*inch}" rpy="${3*M_PI/2} ${M_PI} 0" />
-    <geometry>
-     <mesh filename="package://simplified/meshes/HandleBottom.STL" scale="0.001 0.001 0.001"/>
-    </geometry>
-    </collision>
-    <inertial>
-    <origin xyz="0 -0.07 0.09" rpy="0 0 0" />
-      <mass value="2.03"/>
-      <inertia ixx="0.06" ixy="0" ixz="0" iyy="0.04" iyz="0" izz="0.02"/>
-    </inertial>
- </link>
+    <visual>
+        <origin xyz="0 0 ${21.75*inch}" rpy="${3*M_PI/2} ${M_PI} 0" />
+        <geometry>
+            <mesh filename="package://simplified/meshes/HandleBottom.STL" scale="0.001 0.001 0.001"/>
+        </geometry>
+    </visual>
+    <collision>
+        <origin xyz="0 0 ${21.75*inch}" rpy="${3*M_PI/2} ${M_PI} 0" />
+        <geometry>
+            <mesh filename="package://simplified/meshes/HandleBottom.STL" scale="0.001 0.001 0.001"/>
+        </geometry>
+    </collision>
+    <inertial>
+        <origin xyz="0 -0.07 0.09" rpy="0 0 0" />
+        <mass value="2.03"/>
+        <inertia ixx="0.06" ixy="0" ixz="0" iyy="0.04" iyz="0" izz="0.02"/>
+    </inertial>
+</link>
 <joint name="core_to_bottom_handle_right" type="fixed">
     <parent link="core"/>
@@ -249,25 +267,24 @@
     <origin xyz="${0.75*inch} ${18*inch+(handle_width/2)} 0"/>
   </joint>
+<!-- Handle Right - [HR_L] -->
 <link name="handle_right">
-  <visual>
-    <origin xyz="0 0 ${13.75*inch+handle_height}" rpy="${M_PI/2} 0 ${3*M_PI/2}" />
-    <geometry>
-     <mesh filename="package://simplified/meshes/Handle Revised.STL"
-scale="0.001 0.001 0.001"/>
-    </geometry>
- </visual>
-    <collision>
-    <origin xyz="0 0 ${13.75*inch+handle_height}" rpy="${M_PI/2} 0 ${3*M_PI/2}" />
-    <geometry>
-     <mesh filename="package://simplified/meshes/Handle Revised.STL"
-scale="0.001 0.001 0.001"/>
-    </geometry>
-    </collision>
-    <inertial>
-    <origin xyz="0.02 0.44 0.04" rpy="0 0 0" />
-      <mass value="2.21"/>
-      <inertia ixx="0.48" ixy="0.02" ixz="0" iyy="0.02" iyz="0.02" izz="0.46"/>
-    </inertial>
- </link>
+    <visual>
+        <origin xyz="0 0 ${13.75*inch+handle_height}" rpy="${M_PI/2} 0 ${3*M_PI/2}" />
+        <geometry>
+            <mesh filename="package://simplified/meshes/Handle Revised.STL" scale="0.001 0.001 0.001"/>
+        </geometry>
+    </visual>
+    <collision>
+        <origin xyz="0 0 ${13.75*inch+handle_height}" rpy="${M_PI/2} 0 ${3*M_PI/2}" />
+        <geometry>
+            <mesh filename="package://simplified/meshes/Handle Revised.STL" scale="0.001 0.001 0.001"/>
+        </geometry>
+    </collision>
+    <inertial>
+        <origin xyz="0.02 0.44 0.04" rpy="0 0 0" />
+        <mass value="2.21"/>
+        <inertia ixx="0.48" ixy="0.02" ixz="0" iyy="0.02" iyz="0.02" izz="0.46"/>
+    </inertial>
+</link>
 <joint name="handle_bottom_right_to_handle" type="fixed">
     <parent link="handle_bottom_right"/>
@@ -275,23 +292,24 @@
     <origin xyz="${1.5*inch} ${0*inch} 0"/>
   </joint>
+<!-- Front Right Leg - [FRL_L] -->
 <link name="front_right_leg">
-  <visual>
-    <origin xyz="${2.75*inch-forward_leg_extension} ${0*inch} ${(14.63+1.75)*inch}" rpy="${M_PI/2+0.12} 0 ${-M_PI/2-0.06}" />
-    <geometry>
-     <mesh filename="package://simplified/meshes/Right Front Leg Revised 2.STL" scale="0.001 0.001 0.001"/>
-    </geometry>
- </visual>
-    <collision>
-    <origin xyz="${2.75*inch-forward_leg_extension} ${0*inch} ${(14.63+1.75)*inch}" rpy="${M_PI/2+0.12} 0 ${-M_PI/2-0.06}" />
-    <geometry>
-     <mesh filename="package://simplified/meshes/Right Front Leg Revised 2.STL" scale="0.001 0.001 0.001"/>
-    </geometry>
-    </collision>
-    <inertial>
-    <origin xyz="0.22 -0.14 0.14" rpy="0 0 0"/>
-      <mass value="2.04"/>
-      <inertia ixx="0.08" ixy="-0.06" ixz="0.07" iyy="0.18" iyz="-0.04" izz="0.18"/>
-    </inertial>
- </link>
+    <visual>
+        <origin xyz="${2.75*inch-forward_leg_extension} ${0*inch} ${(14.63+1.75)*inch}" rpy="${M_PI/2+0.12} 0 ${-M_PI/2-0.06}" />
+        <geometry>
+            <mesh filename="package://simplified/meshes/Right Front Leg Revised 2.STL" scale="0.001 0.001 0.001"/>
+        </geometry>
+    </visual>
+    <collision>
+        <origin xyz="${2.75*inch-forward_leg_extension} ${0*inch} ${(14.63+1.75)*inch}" rpy="${M_PI/2+0.12} 0 ${-M_PI/2-0.06}" />
+        <geometry>
+            <mesh filename="package://simplified/meshes/Right Front Leg Revised 2.STL" scale="0.001 0.001 0.001"/>
+        </geometry>
+    </collision>
+    <inertial>
+        <origin xyz="0.22 -0.14 0.14" rpy="0 0 0"/>
+        <mass value="2.04"/>
+        <inertia ixx="0.08" ixy="-0.06" ixz="0.07" iyy="0.18" iyz="-0.04" izz="0.18"/>
+    </inertial>
+</link>
 <joint name="core_to_leg_right_to_front_leg" type="fixed">
     <parent link="core_to_leg_right"/>
@@ -304,23 +322,24 @@
     <origin xyz="${23*inch-forward_leg_extension+backwards_leg_extension} ${4.1*inch} 0"/>
   </joint>
+<!-- Back Right Leg - [BRL_L] -->
 <link name="back_right_leg">
-  <visual>
-    <origin xyz="${backwards_leg_extension} 0 ${17.8*inch}" rpy="0.025 0.41 ${M_PI/2}" />
-    <geometry>
-     <mesh filename="package://simplified/meshes/Right Back Leg Revised 2.STL" scale="0.001 0.001 0.001"/>
-    </geometry>
- </visual>
-    <collision>
-    <origin xyz="0 0 ${17.8*inch}" rpy="0.025 0.41 ${M_PI/2}" />
-    <geometry>
-     <mesh filename="package://simplified/meshes/Right Back Leg Revised 2.STL" scale="0.001 0.001 0.001"/>
-    </geometry>
-    </collision>
-    <inertial>
-    <origin xyz="-0.09 0.03 -0.08" rpy="0 0 0" />
-      <mass value="2.11"/>
-      <inertia ixx="0.04" ixy="-0.01" ixz="0" iyy="0.07" iyz="0" izz="0.04"/>
-    </inertial>
- </link>
+    <visual>
+        <origin xyz="${backwards_leg_extension} 0 ${17.8*inch}" rpy="0.025 0.41 ${M_PI/2}" />
+        <geometry>
+         <mesh filename="package://simplified/meshes/Right Back Leg Revised 2.STL" scale="0.001 0.001 0.001"/>
+        </geometry>
+    </visual>
+    <collision>
+        <origin xyz="0 0 ${17.8*inch}" rpy="0.025 0.41 ${M_PI/2}" />
+        <geometry>
+         <mesh filename="package://simplified/meshes/Right Back Leg Revised 2.STL" scale="0.001 0.001 0.001"/>
+        </geometry>
+    </collision>
+    <inertial>
+        <origin xyz="-0.09 0.03 -0.08" rpy="0 0 0" />
+        <mass value="2.11"/>
+        <inertia ixx="0.04" ixy="-0.01" ixz="0" iyy="0.07" iyz="0" izz="0.04"/>
+    </inertial>
+</link>
 <joint name="back_right_leg_to_wheel" type="continuous">
     <parent link="back_right_leg"/>
@@ -331,23 +350,24 @@
       <joint_properties damping="0.1" friction="0.5"/>
   </joint>
+<!-- Back Right Spinning Wheel - [BRSW_L] -->
 <link name="back_right_spinning_wheel">
-  <visual>
-    <origin xyz="0 0 0" rpy="0 0 ${M_PI}" />
-    <geometry>
-     <mesh filename="package://simplified/meshes/wheel.STL" scale="0.001 0.001 0.001"/>
-    </geometry>
- </visual>
-    <collision>
-    <origin xyz="0 0 0" rpy="0 0 ${M_PI}" />
-    <geometry>
-     <mesh filename="package://simplified/meshes/wheel.STL" scale="0.001 0.001 0.001"/>
-    </geometry>
-    </collision>
-    <inertial>
-    <origin xyz="0 0 0" rpy="0 0 0" />
-      <mass value="2.28"/>
-      <inertia ixx="0.01" ixy="0" ixz="0" iyy="0.02" iyz="0" izz="0.01"/>
-    </inertial>
- </link>
+    <visual>
+        <origin xyz="0 0 0" rpy="0 0 ${M_PI}" />
+        <geometry>
+            <mesh filename="package://simplified/meshes/wheel.STL" scale="0.001 0.001 0.001"/>
+        </geometry>
+    </visual>
+    <collision>
+        <origin xyz="0 0 0" rpy="0 0 ${M_PI}" />
+        <geometry>
+            <mesh filename="package://simplified/meshes/wheel.STL" scale="0.001 0.001 0.001"/>
+        </geometry>
+    </collision>
+    <inertial>
+        <origin xyz="0 0 0" rpy="0 0 0" />
+        <mass value="2.28"/>
+        <inertia ixx="0.01" ixy="0" ixz="0" iyy="0.02" iyz="0" izz="0.01"/>
+    </inertial>
+</link>
 <joint name="back_left_leg_to_wheel" type="continuous">
     <parent link="back_left_leg"/>
@@ -358,23 +378,24 @@
       <joint_properties damping="0.1" friction="0.5"/>
   </joint>
+<!-- Back Left Spinning Wheel - [BLSW_L] -->
 <link name="back_left_spinning_wheel">
-  <visual>
-    <origin xyz="0 0 0" rpy="0 0 ${M_PI}" />
-    <geometry>
-     <mesh filename="package://simplified/meshes/wheel.STL" scale="0.001 0.001 0.001"/>
-    </geometry>
- </visual>
-    <collision>
-   <origin xyz="0 0 0" rpy="0 0 ${M_PI}" />
-    <geometry>
-     <mesh filename="package://simplified/meshes/wheel.STL" scale="0.001 0.001 0.001"/>
-    </geometry>
-    </collision>
-    <inertial>
-    <origin xyz="0 0 0" rpy="0 0 0" />
-      <mass value="2.28"/>
-      <inertia ixx="0.01" ixy="0" ixz="0" iyy="0.02" iyz="0" izz="0.01"/>
-    </inertial>
- </link>
+    <visual>
+        <origin xyz="0 0 0" rpy="0 0 ${M_PI}" />
+        <geometry>
+            <mesh filename="package://simplified/meshes/wheel.STL" scale="0.001 0.001 0.001"/>
+        </geometry>
+    </visual>
+    <collision>
+        <origin xyz="0 0 0" rpy="0 0 ${M_PI}" />
+        <geometry>
+            <mesh filename="package://simplified/meshes/wheel.STL" scale="0.001 0.001 0.001"/>
+        </geometry>
+    </collision>
+    <inertial>
+        <origin xyz="0 0 0" rpy="0 0 0" />
+        <mass value="2.28"/>
+        <inertia ixx="0.01" ixy="0" ixz="0" iyy="0.02" iyz="0" izz="0.01"/>
+    </inertial>
+</link>
 <!-- Front Wheel Yaw Joint Params -->
 <xacro:property name="front_yaw_effort_limit" value="100.0"/>
@@ -398,5 +419,5 @@
     <joint_properties damping="${front_yaw_damping}" friction="${front_yaw_friction}"/>
 </joint>
-<!-- [FRTW_L] -->
+<!-- Front Right Turning Wheel - [FRTW_L] -->
 <link name="front_right_turning_wheel">
   <visual>
@@ -418,5 +439,5 @@
     </inertial>
  </link>
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