Commit message: HUGE REFACTOR - NO FUNCTIONAL CHANGES
- Changes mesh files so that they have origins at the centre of mass
	- ensure that second moments of inertia correspond to the right axes/coordinate system
	- required an overhaul of the urdf

- Made the urdf.xacro file containing the model a lot prettier.
  Now uses xacro features such as:
	- macros
	- includes
	- more macros
	- more properties

- kinect stuff is now in its own xacro file. this file should never change, it is modular
- Slight changes to some names of pieces

File: src/simplified/configs/solidModel.urdf.xacro (robot description, xacro)
@@ -3,37 +3,30 @@
 <origin xyz="0 0 0" rpy="0 0 0"/>
 <!-- Table of Contents - (ctrl-f to jump)
-Xacro Properties:
+Property List:
+    Constants
+    Walker Configuration Dimensions
 Plugins:
-    Wheel Encoders Plugins         [WENC_P]
-    Gazebo Ros Control (Joint Controllers):
-Links:
-    Base Footprint                 [BFP_L]
-    Core (Base Link)               [CORE_L]
-    Front Left Leg                 [FLL_L]
-    Back Left Leg                  [BLL_L]
-    Core to Left Leg (link)        [CTLL_L]
-    Front Left Leg to Back Leg     [FLLTBL_L]
-    Handle Bottom Left             [HBL_L]
-    Handle Left                    [HL_L]
-    Core to Leg Right              [CTLR_L]
-    Handle Bottom Right            [HBR_L]
-    Handle Right                   [HR_L]
-    Front Right Leg                [FRL_L]
-    Back Right Leg                 [BRL_L]
-    Back Right Spinning Wheel      [BRSW_L]
-    Back Left Spinning Wheel       [BLSW_L]
-    Front Right Turning Wheel      [FRTW_L]
-    Front Left Turning Wheel       [FLTW_L]
-    Front Right Spinning Wheel     [FRSW_L]
-    Front Left Spinning Wheel      [FLSW_L]
-    Camera RGB Optical Frame       [CROF_L]
-    Camera Link                    [CAM_L]
+    Gazebo Ros Controls
+    Wheel Encoder
+Links & Joints:
+    Base Coordinate Systems             [BCS]
+    Core                                [CORE]
+    Track Extenders                     [TR_EX]
+    Front Legs                          [FR_LGS]
+    Back Legs                           [BK_LGS]
+    Front Wheels                        [FR_WLS]
+    Back Wheels                         [BK_WLS]
+    Handle Tracks                       [HN_TRS]
+    Handles                             [HNDLS]
+    Kinect Camera                       [KNCT]
 Transmissions:
-    Right Turning Wheel            [RTW_T]
-    Left Turning Wheel             [LTW_T]
-    Right Spinning Wheel           [RSW_T]
-    Left Spinning Wheel            [LSW_T]
-    Back Right Spinning Wheel      [BRSW_T]
-    Back Left Spinning Wheel       [BLSW_T]
+    Right Turning Wheel                 [RTW_T]
+    Left Turning Wheel                  [LTW_T]
+    Right Spinning Wheel                [RSW_T]
+    Left Spinning Wheel                 [LSW_T]
+    Back Right Spinning Wheel           [BRSW_T]
+    Back Left Spinning Wheel            [BLSW_T]
+Physics Params:
+    Wheels (Kp Kd mu1 mu2 etc.)
 -->
 <!-- PROPERTY LIST -->
@@ -41,11 +34,4 @@
 <property name="M_PI" value="3.1415926535897931" />
 <property name="inch" value="0.0254"/>
-<!-- Kinect Camera Module specific properties for pose -->
-<property name="cam_px" value="-0.087" />
-<property name="cam_py" value="-0.0125" />
-<property name="cam_pz" value="0.2870" />
-<property name="cam_or" value="0" />
-<property name="cam_op" value="0" />
-<property name="cam_oy" value="0" />
 <!-- List of Editable Walker Dimensions-->
 <property name="forward_leg_extension" value="${4*inch}" />
@@ -53,5 +39,15 @@
 <property name="frame_width" value="${3*inch}" />
 <property name="handle_width" value="${3*inch}" />
-<property name="handle_height" value="${5*inch}" />
+<property name="extrusion_length" value="0.038" />
+<property name="axle_track" value="${15*inch}" />
+<!-- Just defining wheel base is one thing, however in order to define
+     The position of each wheel w.r.t the position of the core, one must
+     Define both forward and backward wheel extension, and they add up to wheel base
+     Here we define wheel base and backward wheel extension, forward is implicitly defined -->
+<property name="wheel_base" value="0.5" />
+<property name="front_wheel_extension" value="0" />
+<property name="handle_track" value="${20*inch}" />
+<property name="handle_height" value="${43*inch}" />
+<property name="core_width" value="${0.25431 * 2}" />
 <!--    Gazebo Ros Control Plugin
         Allows us to generate controllers for joints
@@ -63,706 +59,294 @@
     </plugin>
 </gazebo>
-<!-- Base Footprint [BFP_L]-->
+<!-- Base Coordinate Systems    :   [BCS]    -->
 <link name="base_footprint">
     <origin xyz="0 0 0" rpy="0 0 0" />
 </link>
+<property name="base_link_height_offset" value="${21.25 * inch}" />
 <joint name="base_joint" type="fixed">
     <parent link="base_footprint"/>
-    <child link="core"/>
-    <origin xyz="0 0 0" rpy="0 0 ${M_PI}" />
-</joint>
-<!-- Core (Base Link) [CORE_L] -->
-<link name="core">
+    <child link="base_link"/>
+    <origin xyz="0 0 ${base_link_height_offset}" rpy="0 0 0" />
+</joint>
+<link name="base_link">
+    <origin xyz="0 0 0" rpy="0 0 0" />
+</link>
+<!-- It would be nice to import things like mass, Ixx Ixy, etc. from a yaml file, or some text file that could be fully or partially generated from solidworks... Unfortunately, there is no support for .yaml files in indigo, but there is in jade, and hopefully that feature will eventually be backported. If it is ever backported, look into grabbing those properties straight form a yaml file)-->
+<xacro:macro name="alink" params="linkName fileName transformXYZ transformRPY mass ixx ixy ixz iyy iyz izz">
+<link name="${linkName}">
     <visual>
-        <origin xyz="0 0 ${31*inch}" rpy="${M_PI/2} ${3*M_PI/2} 0" />
+        <origin xyz="${transformXYZ}" rpy="${transformRPY}"/>
         <geometry>
-            <mesh filename="package://simplified/meshes/Core Revised.STL" scale="0.001 0.001 0.001"/>
+            <mesh filename="${fileName}" scale="0.001 0.001 0.001"/>
         </geometry>
     </visual>
     <collision>
-        <origin xyz="0 0 ${31*inch}" rpy="${M_PI/2} ${3*M_PI/2} 0" />
+        <origin xyz="${transformXYZ}" rpy="${transformRPY}"/>
         <geometry>
-            <mesh filename="package://simplified/meshes/Core Revised.STL" scale="0.001 0.001 0.001"/>
+            <mesh filename="${fileName}" scale="0.001 0.001 0.001"/>
         </geometry>
     </collision>
     <inertial>
-        <origin xyz="0 0.2 -0.2" rpy="0 0 0" />
-        <mass value="7.6"/>
-        <inertia ixx="0.91" ixy="0" ixz="0" iyy="0.47" iyz="-0.37" izz="0.46"/>
+		<origin xyz="${transformXYZ}" rpy="${transformRPY}"/>
+        <mass value="${mass}"/>
+        <inertia ixx="${ixx}" ixy="${ixy}" ixz="${ixz}" iyy="${iyy}" iyz="${iyz}" izz="${izz}" />
     </inertial>
 </link>
-<!-- Front Left Leg - [FLL_L] -->
-<link name="front_left_leg">
-    <visual>
-        <origin xyz="${(-27*inch)-forward_leg_extension} ${-1.6*inch} ${(14.63+1.75)*inch}" rpy="${M_PI/2+0.12} 0 ${-M_PI/2-0.06}" />
-        <geometry>
-            <mesh filename="package://simplified/meshes/Left Front Leg Revised 2.STL" scale="0.001 0.001 0.001"/>
-        </geometry>
-    </visual>
-    <collision>
-        <origin xyz="${(-27*inch)-forward_leg_extension} ${-1.6*inch} ${(14.63+1.75)*inch}" rpy="${M_PI/2+0.12} 0 ${-M_PI/2-0.06}" />
-        <geometry>
-            <mesh filename="package://simplified/meshes/Left Front Leg Revised 2.STL" scale="0.001 0.001 0.001"/>
-        </geometry>
-    </collision>
-    <inertial>
-        <origin xyz="-0.22 -0.13 0.14" rpy="0 0 0" />
-        <mass value="2.04"/>
-        <inertia ixx="0.08" ixy="-0.06" ixz="0.07" iyy="0.18" iyz="-0.04" izz="0.17"/>
-    </inertial>
-</link>
-<!-- Back Left Leg - [BLL_L] -->
-<link name="back_left_leg">
-    <visual>
-        <origin xyz="${backwards_leg_extension} 0 ${17.8*inch}" rpy="0.025 0.41 ${M_PI/2}" />
-        <geometry>
-            <mesh filename="package://simplified/meshes/Back Left Leg Revised 2.STL" scale="0.001 0.001 0.001"/>
-        </geometry>
-    </visual>
-    <collision>
-        <origin xyz="0 0 ${17.8*inch}" rpy="0.025 0.41 ${M_PI/2}" />
-        <geometry>
-            <mesh filename="package://simplified/meshes/Back Left Leg Revised 2.STL" scale="0.001 0.001 0.001"/>
-        </geometry>
-    </collision>
-    <inertial>
-        <origin xyz="-0.09 0.01 -0.08" rpy="0 0 0" />
-        <mass value="2.11"/>
-        <inertia ixx="0.04" ixy="0" ixz="0" iyy="0.07" iyz="0" izz="0.04"/>
-    </inertial>
-</link>
-<!-- Core to Left Leg [CTLL_L] -->
-<link name="core_to_leg_left">
-    <visual>
-        <origin xyz="0 0 ${18.35*inch}" rpy="${M_PI/2} 0 0" />
-        <geometry>
-            <mesh filename="package://simplified/meshes/CoreToLeg.STL" scale="0.001 0.001 0.001"/>
-        </geometry>
-    </visual>
-    <collision>
-        <origin xyz="0 0 ${18.35*inch}" rpy="${M_PI/2} 0 0" />
-        <geometry>
-            <mesh filename="package://simplified/meshes/CoreToLeg.STL" scale="0.001 0.001 0.001"/>
-        </geometry>
-    </collision>
-    <inertial>
-        <origin xyz="0 -0.01 -0.13" rpy="0 0 0" />
-        <mass value="1.56"/>
-        <inertia ixx="0.04" ixy="0" ixz="0" iyy="0.04" iyz="0" izz="0"/>
-    </inertial>
-</link>
-<!-- Front Left Leg to Back Leg [FLLTBL_L] -->
-<joint name="front_left_leg_to_back_leg" type="fixed">
-    <parent link="front_left_leg"/>
-    <child link="back_left_leg"/>
-    <origin xyz="${-6.75*inch-forward_leg_extension+backwards_leg_extension} ${3.9*inch} 0"/>
-</joint>
-<joint name="core_to_leg_left_to_front_leg" type="fixed">
-    <parent link="core_to_leg_left"/>
-    <child link="front_left_leg"/>
-    <origin xyz="${25*inch} ${6.05*inch} 0"/>
-  </joint>
-<joint name="core_to_core_to_leg_left" type="fixed">
+</xacro:macro>
+<xacro:macro name="transmissionMacro" params="tName jointName type">
+<transmission name="${tName}">
+    <type>transmission_interface/SimpleTransmission</type>
+    <joint name="${jointName}">
+        <hardwareInterface>${type}JointInterface</hardwareInterface>
+    </joint>
+    <actuator name="${tName}_actuator">
+        <mechanicalReduction>1</mechanicalReduction>
+        <hardwareInterface>${type}JointInterface</hardwareInterface>
+    </actuator>
+</transmission>
+</xacro:macro>
+<!-- Core   :   [CORE]  -->
+<joint name="link_to_core" type="fixed">
+    <parent link="base_link"/>
+    <child link="core"/>
+    <origin xyz="0 ${-0.5 * core_width} 0" rpy="0 0 0" />
+</joint>
+<xacro:alink
+    linkName="core"
+    fileName="package://simplified/meshes/Core.STL"
+    transformXYZ="0.02504 ${0.5 * core_width} 0.01849"
+    transformRPY="0 0 0"
+    mass="7.6"
+    ixx="0.91" ixy="0" ixz="0" iyy="0.47" iyz="-0.37" izz="0.46"
+/>
+<!-- Track Extenders    :   [TR_EX] -->
+<property name="track_extender_wheel_offset" value="${2.7*inch}" />
+<property name="track_extender_padding_thickness" value="0.00955" />
+<xacro:macro name="trackExtender" params="prefix reflect rotate">
+<xacro:alink
+    linkName="track_extender_${prefix}"
+    fileName="package://simplified/meshes/CoreToLeg.STL"
+    transformXYZ="-0.0057 ${0.06219 * reflect} 0.027"
+    transformRPY="0 0 ${rotate*M_PI}"
+    mass="1.56"
+    ixx="0.03" ixy="0" ixz="0" iyy="0" iyz="0" izz="0.3"
+/>
+</xacro:macro>
+<xacro:trackExtender prefix="right" reflect =  "1" rotate="0"/>
+<xacro:trackExtender prefix="left"  reflect = "-1" rotate="1"/>
+<joint name="core_to_right_track_extender" type="fixed">
     <parent link="core"/>
-    <child link="core_to_leg_left"/>
-    <origin xyz="${0.65*inch} ${-4*inch-(frame_width/2)} 0"/>
-  </joint>
-<!-- Handle Bottom Left - [HBL_L] -->
-<link name="handle_bottom_left">
-    <visual>
-        <origin xyz="0 0 ${21.75*inch}" rpy="${M_PI/2} 0 0" />
-        <geometry>
-            <mesh filename="package://simplified/meshes/HandleBottom.STL" scale="0.001 0.001 0.001"/>
-        </geometry>
-    </visual>
-    <collision>
-        <origin xyz="0 0 ${21.75*inch}" rpy="${M_PI/2} 0 0" />
-        <geometry>
-            <mesh filename="package://simplified/meshes/HandleBottom.STL" scale="0.001 0.001 0.001"/>
-        </geometry>
-    </collision>
-    <inertial>
-        <origin xyz="0 0.07 0.09" rpy="0 0 0" />
-        <mass value="0.5"/>
-        <inertia ixx="0.06" ixy="0" ixz="0" iyy="0.04" iyz="0" izz="0.02"/>
-    </inertial>
-</link>
-<joint name="core_to_bottom_handle_left" type="fixed">
+    <child link="track_extender_right"/>
+    <origin xyz="0 ${-0.5 * (axle_track - core_width)} ${-2 * (track_extender_padding_thickness + extrusion_length)}"/>
+</joint>
+<joint name="core_to_left_track_extender" type="fixed">
     <parent link="core"/>
-    <child link="handle_bottom_left"/>
-    <origin xyz="${0.7*inch} ${-2*inch-(handle_width/2)} 0"/>
-  </joint>
-<!-- Handle Left - [HL_L] -->
-<link name="handle_left">
-  <visual>
-    <origin xyz="0 0 ${13.75*inch+handle_height}" rpy="${M_PI/2} 0 ${3*M_PI/2}" />
-    <geometry>
-     <mesh filename="package://simplified/meshes/Handle Revised.STL" scale="0.001 0.001 0.001"/>
-    </geometry>
- </visual>
-    <collision>
-   <origin xyz="0 0 ${13.75*inch+handle_height}" rpy="${M_PI/2} 0 ${3*M_PI/2}" />
-    <geometry>
-     <mesh filename="package://simplified/meshes/Handle Revised.STL" scale="0.001 0.001 0.001"/>
-    </geometry>
-    </collision>
-    <inertial>
-    <origin xyz="0.02 0.44 0.04" rpy="0 0 0" />
-      <mass value="2.21"/>
-      <inertia ixx="0.48" ixy="0.02" ixz="0" iyy="0.02" iyz="0.02" izz="0.46"/>
-    </inertial>
- </link>
-<joint name="handle_bottom_left_to_handle" type="fixed">
-    <parent link="handle_bottom_left"/>
-    <child link="handle_left"/>
-    <origin xyz="${1.5*inch} ${1.5*inch} 0"/>
-  </joint>
-<!-- Core to Leg Right - [CTLR_L] -->
-<link name="core_to_leg_right">
-    <visual>
-        <origin xyz="0 0 ${18.35*inch}" rpy="${3*M_PI/2} ${M_PI} 0" />
-        <geometry>
-            <mesh filename="package://simplified/meshes/CoreToLeg.STL" scale="0.001 0.001 0.001"/>
-        </geometry>
-    </visual>
-    <collision>
-        <origin xyz="0 0 ${18.35*inch}" rpy="${3*M_PI/2} ${M_PI} 0" />
-        <geometry>
-            <mesh filename="package://simplified/meshes/CoreToLeg.STL" scale="0.001 0.001 0.001"/>
-        </geometry>
-    </collision>
-    <inertial>
-        <origin xyz="0 -0.11 -0.02" rpy="0 0 0" />
-        <mass value="1.56"/>
-        <inertia ixx="0.03" ixy="0" ixz="0" iyy="0" iyz="0" izz="0.3"/>
-    </inertial>
-</link>
-<joint name="core_to_core_to_leg_right" type="fixed">
+    <child link="track_extender_left"/>
+    <origin xyz="0 ${1 * core_width + 0.5 * (axle_track - core_width)} ${-2 * (track_extender_padding_thickness + extrusion_length)}"/>
+</joint>
+<!-- Front Legs     :   [FR_LGS]    -->
+<property name="front_leg_length" value="0.399108" />
+<xacro:macro name="trackExtenderToFrontLegJoint" params="prefix">
+<joint name="track_extender_to_front_leg_${prefix}" type="fixed">
+    <parent link="track_extender_${prefix}"/>
+    <child link="front_${prefix}_leg"/>
+    <origin xyz="${0.2 + front_wheel_extension - front_leg_length} 0 0"/>
+</joint>
+</xacro:macro>
+<xacro:trackExtenderToFrontLegJoint prefix="right"/>
+<xacro:trackExtenderToFrontLegJoint prefix="left"/>
+<xacro:alink
+    linkName="front_right_leg"
+    fileName="package://simplified/meshes/Left Front Leg.STL"
+    transformXYZ="0.22295 -0.00299 -0.03424"
+    transformRPY="0 0 ${M_PI / -2}"
+    mass="2.04"
+    ixx="0.08" ixy="-0.06" ixz="0.07" iyy="0.18" iyz="-0.04" izz="0.17"
+/>
+<xacro:alink
+    linkName="front_left_leg"
+    fileName="package://simplified/meshes/Right Front Leg.STL"
+    transformXYZ="0.22295 0.00299 -0.03424"
+    transformRPY="0 0 0"
+    mass="2.04"
+    ixx="0.08" ixy="-0.06" ixz="0.07" iyy="0.18" iyz="-0.04" izz="0.18"
+/>
+<!-- Back Legs      :   [BK_LGS] -->
+<property name="back_leg_length" value="0.300" />
+<property name="back_leg_tip_to_over_wheel_offset" value="0" />
+<xacro:macro name="frontToBackLegJoint" params="prefix">
+<joint name="${prefix}_front_to_back_leg" type="fixed">
+    <parent link="front_${prefix}_leg"/>
+    <child link="back_${prefix}_leg"/>
+    <origin xyz="${back_leg_length - (wheel_base - front_leg_length) - back_leg_tip_to_over_wheel_offset} 0 ${-1 * extrusion_length}"/>
+</joint>
+</xacro:macro>
+<xacro:frontToBackLegJoint prefix="right"/>
+<xacro:frontToBackLegJoint prefix="left"/>
+<xacro:alink
+    linkName="back_right_leg"
+    fileName="package://simplified/meshes/Left Back Leg.STL"
+    transformXYZ="-0.1947 -0.00554 -0.06712"
+    transformRPY="0 0 ${M_PI/-2}"
+    mass="2.11"
+    ixx="0.04" ixy="0" ixz="0" iyy="0.07" iyz="0" izz="0.04"
+/>
+<xacro:alink
+    linkName="back_left_leg"
+    fileName="package://simplified/meshes/Right Back Leg.STL"
+    transformXYZ="-0.1947 0.00554 -0.06712"
+    transformRPY="0 0 0"
+    mass="2.11"
+    ixx="0.04" ixy="0" ixz="0" iyy="0.07" iyz="0" izz="0.04"
+/>
+<!-- Front Wheels           [FR_WLS]  -->
+<property name="front_wheel_rotation_joint_offset" value="0.000" />
+<property name="front_wheel_carriage_to_axle_z_offset" value ="-0.14" />
+<property name="front_wheel_carriage_to_axle_x_offset" value ="-0.075" />
+<xacro:macro name="frontwheelassembly" params="prefix reflect">
+<!-- Wheel Carriage (Yaw)-->
+<joint name="${prefix}_front_leg_to_wheel_carriage" type="continuous">
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